File: KiCAD/FreeDSP_SMD_AB.sch (KiCad schematic (older format))
At the start: 194 parts, among them IC1 ADAU1701, IC2 24AA256, IC3 24AA256, J1 Conn_01x06, J10 Conn_02x08_Odd_Even, J2 Conn_Coaxial, J3 Conn_02x10_Odd_Even, J4 Conn_Coaxial, J5 Conn_Coaxial, J6 Conn_Coaxial, J7 Conn_Coaxial, J8 Conn_Coaxial, J9 Conn_Coaxial_Power, P1 USBi, Q1 2SC3326, Q10 IRLML6402, Q2 2N7002, Q3 2SC3326, Q4 2N7002, Q5 2SC3326, Q7 2SC3326, Q8 2SB1203, SW1 SW_SPDT, U1 LME49720, U2 74LV541A, U3 LME49720, U4 LME49720, U5 LME49720, U6 AZ1117-ADJ, U7 AZ1117-ADJ, X1 12.288MHz

Commit message: Add files via upload
Other:
- note added: "(2nd LEFT)"
- note added: "(2nd RIGHT)"
- note added: "(LEFT)"
- note added: "(PRI-LEFT)"
- note added: "(PRI-RIGHT)"
- note added: "(RIGHT)"
Changed lines of the file:
@@
 Title "FreeDSP AUAU1701 A/B Switchable Audio Board "
 Date "2019-04-20"
-Rev "0.4"
+Rev "0.41"
 Comp "CyberPit HILO"
 Comment1 "https://cyberpithilo.web.fc2.com/"
@@
 	1    0    0    -1
 $EndComp
-Text Notes 875  4675 0    50   ~ 10
+Text Notes 900  5925 0    50   ~ 10
 INPUT 0
 Wire Notes Line
-	875  4700 875  4575
+	900  5950 900  5825
 Wire Notes Line
-	1200 4700 1200 4575
+	1225 5950 1225 5825
 Wire Notes Line
-	900  5925 900  5800
+	875  4700 875  4575
 Wire Notes Line
-	1225 5925 1225 5800
+	1200 4700 1200 4575
 Wire Notes Line
-	900  5925 1225 5925
+	875  4700 1200 4700
 Wire Notes Line
-	875  4575 1200 4575
+	900  5825 1225 5825
 Wire Notes Line
-	875  4700 1200 4700
-Text Notes 900  5900 0    50   ~ 10
+	900  5950 1225 5950
+Text Notes 875  4675 0    50   ~ 10
 INPUT 1
 Wire Notes Line
-	900  5800 1225 5800
+	875  4575 1200 4575
 Text Notes 15475 1900 0    50   ~ 10
 OUTPUT0
@@
 Text Notes 3625 1275 0    50   Italic 0
 Use Si Switching Diode for D1\nShotkey is NOT suitable
+Text Notes 875  4825 0    50   ~ 0
+(RIGHT)
+Text Notes 925  6075 0    50   ~ 0
+(LEFT)
+Text Notes 15425 4000 0    50   ~ 0
+(PRI-RIGHT)
+Text Notes 15450 2050 0    50   ~ 0
+(PRI-LEFT)
+Text Notes 15425 8075 0    50   ~ 0
+(2nd RIGHT)
+Text Notes 15425 6050 0    50   ~ 0
+(2nd LEFT)
 $EndSCHEMATC

Commit message: Add files via upload
Parts:
- R49: value 47k -> 4.7k
Other:
- note added: "Fixed: R49 vlalue to 4.7k"
- note removed: "(2nd LEFT)"
- note removed: "(2nd RIGHT)"
- note removed: "(LEFT)"
- note removed: "(PRI-LEFT)"
- note removed: "(PRI-RIGHT)"
- note removed: "(RIGHT)"
Changed lines of the file:
@@
 EESchema Schematic File Version 4
-LIBS:FreeDSP_SMD_AB-cache
-EELAYER 29 0
+EELAYER 30 0
 EELAYER END
 $Descr A3 16535 11693
 encoding utf-8
 Sheet 1 1
-Title "FreeDSP AUAU1701 A/B Switchable Audio Board "
-Date "2019-04-20"
-Rev "0.41"
+Title "FreeDSP Classic SMD A/B "
+Date "2020-11-22"
+Rev "0.42"
 Comp "CyberPit HILO"
 Comment1 "https://cyberpithilo.web.fc2.com/"
@@
 P 4675 7175
 F 0 "R49" V 4755 7175 40  0000 C CNN
-F 1 "47k" V 4675 7175 40  0000 C CNN
+F 1 "4.7k" V 4675 7175 40  0000 C CNN
 F 2 "Resistors_SMD:R_0805_HandSoldering" V 4605 7175 30  0001 C CNN
 F 3 "~" H 4675 7175 30  0000 C CNN
@@
 	1    0    0    -1
 $EndComp
-Text Notes 900  5925 0    50   ~ 10
+Text Notes 875  4675 0    50   ~ 10
 INPUT 0
 Wire Notes Line
-	900  5950 900  5825
-Wire Notes Line
-	1225 5950 1225 5825
-Wire Notes Line
 	875  4700 875  4575
 Wire Notes Line
 	1200 4700 1200 4575
 Wire Notes Line
-	875  4700 1200 4700
+	900  5925 900  5800
 Wire Notes Line
-	900  5825 1225 5825
+	1225 5925 1225 5800
 Wire Notes Line
-	900  5950 1225 5950
-Text Notes 875  4675 0    50   ~ 10
-INPUT 1
+	900  5925 1225 5925
 Wire Notes Line
 	875  4575 1200 4575
+Wire Notes Line
+	875  4700 1200 4700
+Text Notes 900  5900 0    50   ~ 10
+INPUT 1
+Wire Notes Line
+	900  5800 1225 5800
 Text Notes 15475 1900 0    50   ~ 10
 OUTPUT0
@@
 Text Notes 3625 1275 0    50   Italic 0
 Use Si Switching Diode for D1\nShotkey is NOT suitable
-Text Notes 875  4825 0    50   ~ 0
-(RIGHT)
-Text Notes 925  6075 0    50   ~ 0
-(LEFT)
-Text Notes 15425 4000 0    50   ~ 0
-(PRI-RIGHT)
-Text Notes 15450 2050 0    50   ~ 0
-(PRI-LEFT)
-Text Notes 15425 8075 0    50   ~ 0
-(2nd RIGHT)
-Text Notes 15425 6050 0    50   ~ 0
-(2nd LEFT)
+Text Notes 4950 6475 3    50   Italic 0
+Fixed: R49 vlalue to 4.7k
 $EndSCHEMATC
